Commit message: Add camera and lidar

File: description/camera.xacro (robot description, xacro)
@@ -4,12 +4,13 @@
         <parent link="chassis"/>
         <child link="camera_link"/>
-        <origin xyz="0.425 0 0.08" rpy="0 0 0"/>
+        <origin xyz="0.35 0 0.08" rpy="0 0 0"/>
     </joint>
     <link name="camera_link">
         <visual>
             <geometry>
-                <box size="0.010 0.03 0.03"/>
+                <mesh filename="file:///home/artem/mesh_car/src/mesh_car/meshes/camera.stl" scale="0.0025 0.0025 0.0025"/>
+                <!-- <box size="0.010 0.03 0.03"/> -->
             </geometry>
-            <material name="red"/>
+            <material name="blue"/>
         </visual>
     </link>
@@ -21,5 +22,5 @@
     <link name="camera_link_optical"></link>
     <gazebo reference="camera_link">
-        <material>Gazebo/Red</material>
+        <material>Gazebo/Blue</material>
         <sensor name="camera" type="camera">
             <pose> 0 0 0 0 0 0 </pose>
@@ -34,5 +35,5 @@
                 </image>
                 <clip>
-                    <near>0.05</near>
+                    <near>0.1</near>
                     <far>8.0</far>
                 </clip>

File: description/gazebo_control.xacro (robot description, xacro)
@@ -12,9 +12,9 @@
             <wheel_separation>0.35</wheel_separation>
             <wheel_separation>0.35</wheel_separation>
-            <wheel_diameter>0.05</wheel_diameter>
-            <wheel_diameter>0.05</wheel_diameter>
+            <wheel_diameter>0.035</wheel_diameter>
+            <wheel_diameter>0.035</wheel_diameter>
             <!-- Limits -->
-            <max_wheel_torque>20</max_wheel_torque>
-            <max_wheel_acceleration>2.0</max_wheel_acceleration>
+            <max_wheel_torque>50</max_wheel_torque>
+            <max_wheel_acceleration>10.0</max_wheel_acceleration>
             <!-- Output -->
             <odometry_frame>odom</odometry_frame>

File: description/lidar.xacro (robot description, xacro)
@@ -4,10 +4,10 @@
         <parent link="chassis"/>
         <child link="laser_frame"/>
-        <origin xyz="0.1 0 0.175" rpy="0 0 0"/>
+        <origin xyz="0.075 0 0.14" rpy="0 0 0"/>
     </joint>
     <link name="laser_frame">
         <visual>
             <geometry>
-                <cylinder radius="0.05" length="0.04"/>
+                <mesh filename="file:///home/artem/mesh_car/src/mesh_car/meshes/lidar.stl" scale="0.0015 0.0015 0.0015"/>
             </geometry>
             <material name="red"/>

File: description/robot_core.xacro (robot description, xacro)
@@ -28,5 +28,5 @@
     <link name="chassis">
         <visual>
-            <origin xyz="0.1 0 0.025" rpy="0 0 ${pi/2}"/>
+            <origin xyz="0.1 0 -0.025" rpy="0 0 ${pi/2}"/>
             <geometry>
                <mesh filename="file:///home/artem/mesh_car/src/mesh_car/meshes/car.stl" scale="0.005 0.005 0.005"/>
@@ -53,5 +53,5 @@
         <parent link="base_link"/>
         <child link="left_wheel"/>
-        <origin xyz="-0.115 0.15 0.03" rpy="0 0 0" />
+        <origin xyz="-0.115 0.15 0" rpy="0 0 0" />
         <axis xyz="0 1 0"/>
     </joint>
@@ -81,5 +81,5 @@
         <parent link="base_link"/>
         <child link="left2_wheel"/>
-        <origin xyz="0.285 0.15 0.03" rpy="0 0 0" />
+        <origin xyz="0.285 0.15 0" rpy="0 0 0" />
         <axis xyz="0 1 0"/>
     </joint>
@@ -109,5 +109,5 @@
         <parent link="base_link"/>
         <child link="right_wheel"/>
-        <origin xyz="-0.115 -0.15 0.03" rpy="0 0 0" />
+        <origin xyz="-0.115 -0.15 0" rpy="0 0 0" />
         <axis xyz="0 -1 0"/>
     </joint>
@@ -137,5 +137,5 @@
         <parent link="base_link"/>
         <child link="right2_wheel"/>
-        <origin xyz="0.285 -0.15 0.03" rpy="0 0 0" />
+        <origin xyz="0.285 -0.15 0" rpy="0 0 0" />
         <axis xyz="0 -1 0"/>
     </joint>

Commit message: Improved robot + add sonar

File: description/camera.xacro (robot description, xacro)
@@ -12,5 +12,5 @@
                 <!-- <box size="0.010 0.03 0.03"/> -->
             </geometry>
-            <material name="blue"/>
+            <material name="grey"/>
         </visual>
     </link>
@@ -22,8 +22,8 @@
     <link name="camera_link_optical"></link>
     <gazebo reference="camera_link">
-        <material>Gazebo/Blue</material>
+        <material>Gazebo/Grey</material>
         <sensor name="camera" type="camera">
             <pose> 0 0 0 0 0 0 </pose>
-            <visualize>true</visualize>
+            <visualize>false</visualize>
             <update_rate>10</update_rate>
             <camera>
@@ -35,5 +35,5 @@
                 </image>
                 <clip>
-                    <near>0.1</near>
+                    <near>0.3</near>
                     <far>8.0</far>
                 </clip>

File: description/gazebo_control.xacro (robot description, xacro)
@@ -5,8 +5,8 @@
             <!-- Wheel Information -->
             <num_wheel_pairs>2</num_wheel_pairs>
-            <left_joint>left_wheel_joint</left_joint>
-            <left_joint>left2_wheel_joint</left_joint>
-            <right_joint>right_wheel_joint</right_joint>
-            <right_joint>right2_wheel_joint</right_joint>
+            <left_joint>left_rare_wheel_joint</left_joint>
+            <left_joint>left_front_wheel_joint</left_joint>
+            <right_joint>right_rare_wheel_joint</right_joint>
+            <right_joint>right_front_wheel_joint</right_joint>
             <!-- Kinematics -->
             <wheel_separation>0.35</wheel_separation>
@@ -29,12 +29,11 @@
         <plugin name="diff_drive_joint_states" filename="libgazebo_ros_joint_state_publisher.so">
             <ros>
-                <!-- <namespace>/br</namespace> -->
                 <remapping>~/out:=joint_states</remapping>
             </ros>
             <update_rate>50</update_rate>
-            <joint_name>left_wheel_joint</joint_name>
-            <joint_name>left2_wheel_joint</joint_name>
-            <joint_name>right_wheel_joint</joint_name>
-            <joint_name>right2_wheel_joint</joint_name>
+            <left_joint>left_rare_wheel_joint</left_joint>
+            <left_joint>left_front_wheel_joint</left_joint>
+            <right_joint>right_rare_wheel_joint</right_joint>
+            <right_joint>right_front_wheel_joint</right_joint>
         </plugin>
     </gazebo>

File: description/lidar.xacro (robot description, xacro)
@@ -11,5 +11,5 @@
                 <mesh filename="file:///home/artem/mesh_car/src/mesh_car/meshes/lidar.stl" scale="0.0015 0.0015 0.0015"/>
             </geometry>
-            <material name="red"/>
+            <material name="white"/>
         </visual>
         <collision>
@@ -23,9 +23,10 @@
     </link>
     <gazebo reference="laser_frame">
-        <material>Gazebo/Red</material>
+        <material>Gazebo/White</material>
         <sensor name="laser" type="ray">
             <pose> 0 0 0 0 0 0 </pose>
-            <visualize>false</visualize>
-            <update_rate>10</update_rate>
+            <always_on>true</always_on>
+            <visualize>true</visualize>
+            <update_rate>20</update_rate>
             <ray>
                 <scan>
@@ -35,4 +36,16 @@
                         <max_angle>3.14</max_angle>
                     </horizontal>
+                    <!-- <horizontal>
+                            <samples>20</samples>
+                            <resolution>1</resolution>
+                            <min_angle>${-pi/90}</min_angle>
+                            <max_angle>${pi/90}</max_angle>
+                        </horizontal>
+                        <vertical>
+                            <samples>20</samples>
+                            <resolution>1</resolution>
+                            <min_angle>${-pi/150}</min_angle>
+                            <max_angle>${pi/150}</max_angle>
+                        </vertical> -->
                 </scan>
                 <range>

File: description/robot.urdf.xacro (robot description, xacro)
@@ -3,5 +3,6 @@
     <xacro:include filename="robot_core.xacro" />
     <xacro:include filename="gazebo_control.xacro"/>
-    <xacro:include filename="lidar.xacro"/>
+    <!-- <xacro:include filename="lidar.xacro"/> -->
+    <xacro:include filename="sonar.xacro"/>
     <xacro:include filename="camera.xacro"/>
 </robot>

File: description/robot_core.xacro (robot description, xacro)
@@ -11,4 +11,7 @@
         <color rgba="1 0.3 0.1 1"/>
     </material>
+    <material name="grey">
+        <color rgba="0.5 0.5 0.5 1"/>
+    </material>
     <material name="blue">
         <color rgba="0.2 0.2 1 1"/>
@@ -19,4 +22,12 @@
     <!-- BASE LINK -->
     <link name="base_link">
+    </link>
+     <!-- BASE_FOOTPRINT LINK -->
+    <joint name="base_footprint_joint" type="fixed">
+        <parent link="base_link"/>
+        <child link="base_footprint"/>
+        <origin xyz="0 0 0" rpy="0 0 0"/>
+    </joint>
+    <link name="base_footprint">
     </link>
     <!-- CHASSIS LINK -->
@@ -32,5 +43,5 @@
                <mesh filename="file:///home/artem/mesh_car/src/mesh_car/meshes/car.stl" scale="0.005 0.005 0.005"/>
             </geometry>
-            <material name="white"/>
+            <material name="orange"/>
         </visual>
         <collision>
@@ -46,20 +57,20 @@
     <gazebo reference="chassis">
         <material>
-            Gazebo/White
+            Gazebo/Orange
         </material>
     </gazebo>
     <!-- LEFT WHEEL LINK -->
-    <joint name="left_wheel_joint" type="continuous">
+    <joint name="left_rare_wheel_joint" type="continuous">
         <parent link="base_link"/>
-        <child link="left_wheel"/>
+        <child link="left_rare_wheel"/>
         <origin xyz="-0.115 0.15 0" rpy="0 0 0" />
         <axis xyz="0 1 0"/>
     </joint>
-    <link name="left_wheel">
+    <link name="left_rare_wheel">
         <visual>
             <geometry>
                 <mesh filename="file:///home/artem/mesh_car/src/mesh_car/meshes/left_tire.stl" scale="0.002 0.002 0.002"/>
             </geometry>
-            <material name="blue"/>
+            <material name="black"/>
         </visual>
         <collision>
@@ -72,22 +83,22 @@
         </xacro:inertial_cylinder>
     </link>
-    <gazebo reference="left_wheel">
+    <gazebo reference="left_rare_wheel">
         <material>
-            Gazebo/Blue
+            Gazebo/Black
         </material>
     </gazebo>
     <!-- LEFT2 WHEEL LINK -->
-    <joint name="left2_wheel_joint" type="continuous">
+    <joint name="left_front_wheel_joint" type="continuous">
         <parent link="base_link"/>
-        <child link="left2_wheel"/>
+        <child link="left_front_wheel"/>
         <origin xyz="0.285 0.15 0" rpy="0 0 0" />
         <axis xyz="0 1 0"/>
     </joint>
-    <link name="left2_wheel">
+    <link name="left_front_wheel">
         <visual>
             <geometry>
                  <mesh filename="file:///home/artem/mesh_car/src/mesh_car/meshes/left_tire.stl" scale="0.002 0.002 0.002"/>
             </geometry>
-            <material name="blue"/>
+            <material name="black"/>
         </visual>
         <collision>
@@ -100,22 +111,22 @@
         </xacro:inertial_cylinder>
     </link>
-    <gazebo reference="left2_wheel">
+    <gazebo reference="left_front_wheel">
         <material>
-            Gazebo/Blue
+            Gazebo/Black
         </material>
     </gazebo>
     <!-- RIGHT WHEEL LINK -->
-    <joint name="right_wheel_joint" type="continuous">
+    <joint name="right_rare_wheel_joint" type="continuous">
         <parent link="base_link"/>
-        <child link="right_wheel"/>
+        <child link="right_rare_wheel"/>
         <origin xyz="-0.115 -0.15 0" rpy="0 0 0" />
         <axis xyz="0 -1 0"/>
     </joint>
-    <link name="right_wheel">
+    <link name="right_rare_wheel">
         <visual>
             <geometry>
                 <mesh filename="file:///home/artem/mesh_car/src/mesh_car/meshes/right_tire.stl" scale="0.002 0.002 0.002"/>
             </geometry>
-            <material name="blue"/>
+            <material name="black"/>
         </visual>
         <collision>
@@ -128,22 +139,22 @@
         </xacro:inertial_cylinder>
     </link>
-     <gazebo reference="right_wheel">
+     <gazebo reference="right_rare_wheel">
         <material>
-            Gazebo/Blue
+            Gazebo/Black
         </material>
     </gazebo>
     <!-- RIGHT2 WHEEL LINK -->
-    <joint name="right2_wheel_joint" type="continuous">
+    <joint name="right_front_wheel_joint" type="continuous">
         <parent link="base_link"/>
-        <child link="right2_wheel"/>
+        <child link="right_front_wheel"/>
         <origin xyz="0.285 -0.15 0" rpy="0 0 0" />
         <axis xyz="0 -1 0"/>
     </joint>
-    <link name="right2_wheel">
+    <link name="right_front_wheel">
         <visual>
             <geometry>
                 <mesh filename="file:///home/artem/mesh_car/src/mesh_car/meshes/right_tire.stl" scale="0.002 0.002 0.002"/>
             </geometry>
-            <material name="blue"/>
+            <material name="black"/>
         </visual>
         <collision>
@@ -156,7 +167,7 @@
         </xacro:inertial_cylinder>
     </link>
-     <gazebo reference="right2_wheel">
+     <gazebo reference="right_front_wheel">
         <material>
-            Gazebo/Blue
+            Gazebo/Black
         </material>
     </gazebo>
